File: PCB/hackpad again.kicad_pcb (KiCad board)
At the start: 2 copper layers, 50 x 59.3 mm, 7 parts, among them U1 Seeed_Studio_XIAO_Series_XIAO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

Commit message: ..
Parts:
- moved PB2 1.37 mm to (161.1, 109.5)
- moved PB1 1.14 mm to (142.1, 109.5)
- moved PB4 0.64 mm to (161.1, 128.6)
Routing:
- net GND: track 122.3 -> 124.1 mm
- net U1_11: track 44.1 -> 45.6 mm
- net U1_8: track 17.2 -> 18.3 mm
- net U1_10: track 55.9 -> 55.3 mm
Other:
- outline, holes or cut-outs redrawn
